File: Hardware/SST-SCB/SST-SCB.kicad_sch (KiCad schematic)
At the start: 13 parts, among them J1 MJ-179PH, J2 Conn_01x03_Pin, J3 Conn_01x04_Pin, Q1 2SJ498-D, U1 FT231XS_Breakout, U2 LT1785AxN8

Commit message: Commit Serial Servo Tester for Servo Control Board
Parts:
- removed D1: 11EQS03L, Diode_THT:D_T-1_P10.16mm_Horizontal, symbol Device:D_Schottky
- removed J2: Conn_01x03_Pin, Connector_PinHeader_2.54mm:PinHeader_1x03_P2.54mm_Horizontal, symbol Connector:Conn_01x03_Pin
- removed J3: Conn_01x04_Pin, Connector_JST:JST_EH_S4B-EH_1x04_P2.50mm_Horizontal, symbol Connector:Conn_01x04_Pin
- removed Q1: 2SJ498-D, Package_TO_SOT_THT:TO-92S_Wide, symbol Simulation_SPICE:PJFET
- removed R2: 5.1k, Resistor_THT:R_Axial_DIN0207_L6.3mm_D2.5mm_P10.16mm_Horizontal, symbol Device:R
- removed TH1: PTGL07AR820M9A51B0, Capacitor_THT:C_Disc_D8.0mm_W5.0mm_P5.00mm, symbol Device:Thermistor_PTC
- added C1: C, Capacitor_THT:C_Radial_D8.0mm_H11.5mm_P3.50mm, symbol Device:C
- added J25: Conn_01x02_Pin, Connector_JST:JST_VH_B2P-VH_1x02_P3.96mm_Vertical, symbol Connector:Conn_01x02_Pin
- renumbered J1 to J27
Connections:
- net GND: now also C1.2, J25.2 (Pin_2)
- net VCC: now also C1.1, J25.1 (Pin_1)
- net at R4.2: now also R1.2, R3.2, U1.1 (5V), U1.3 (VCCIO), U2.8 (VCC)
- net ~{EN_4PIN}: no longer names the net of U1.9 (CBUS3)
- no-connect marks 10 -> 11
Other:
- added sheet Servo Port (servo_port.kicad_sch)
- moved on the sheet: J27
