File: SST-SCB/SST-SCB.kicad_pcb (KiCad board)
At the start: 2 copper layers, 42 x 55 mm, 37 parts, among them J1 Conn_01x03_Pin, J10 Conn_01x03_Pin, J11 Conn_01x03_Pin, J12 Conn_01x03_Pin, J13 Conn_01x03_Pin, J14 Conn_01x03_Pin, J15 Conn_01x03_Pin, J16 Conn_01x03_Pin, J17 Conn_01x03_Pin, J18 Conn_01x03_Pin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

Commit message: Fix PCB patterns
Other:
- board text added: "G V S"
- board text added: "S V G"
